File: PCB Files/Passthrough_HarnessBox_Final.kicad_pcb (KiCad board)
At the start: 4 copper layers, 82 x 43 mm, 20 parts, among them J1 JAE DX07S024XJ1R1100, J2 Molex 2125280400, J3 JAE MX34032NF4, J4 JAE MX34032NF4, K1 G5V-2 DC12, Q1 DMN3200U-7, U1 Vishay DG419LEDY-T1-GE4, U2 Vishay DG419LEDY-T1-GE4

Commit message: Change K1 to Omron G5V-2-H1 DC12 (high-sensitivity coil)
K1's coil is hard-tied across VIN/GND, so it is energized continuously
whenever the box is powered and sees the raw automotive rail. The
standard G5V-2 DC12 is rated 120% max coil voltage = 14.4 V, which a
running alternator rail sits right on top of. The high-sensitivity -H1
variant is rated 180% max = 21.6 V and drops the coil from
288 ohm / 41.7 mA / ~500 mW to 960 ohm / 12.5 mA / ~150 mW, which also
removes ~29 mA of permanent quiescent draw and cuts the coil
self-heating that Omron's "Long-term Continuously ON Contacts"
precaution warns about.

Pick-up (9.0 V) and drop-out (0.6 V) are unchanged, so the fail-safe
thresholds are identical. Accepted trade-offs: max switching current
2 A -> 1 A and contact resistance 50 -> 100 mOhm max (both far inside
spec for camera/VCU signal pairs), and shock malfunction rating
200 -> 100 m/s2.

The -H1 is package- and pin-identical to the G5V-2 (20.5 x 10.1 x
11.5 mm, 7.62/5.08/5.08 pitch, 7.62 mm row spacing, eight 1 mm holes),
verified against the Omron datasheet drawing, so no pad, track, zone or
3D model changed. Footprint renamed to My_Components:Omron
G5V-2-H1-DC12; MPN and LCSC part (C128021) added to the schematic
symbol as well as the footprint, since footprint-only fields are
discarded by the next Update PCB from Schematic.

Also corrects the design review, which still described a Panasonic
TQ2-12V in this position and claimed the NO throws were unwired. They
are not: each pole's common is the VCU side (4/13), NC is the CAMERA
side (6/11), and NO (8/9) feeds the DG419 analog switches.

Co-Authored-By: Claude Opus 5 <noreply@anthropic.com>
Parts:
- K1: value G5V-2 DC12 -> G5V-2-H1 DC12; footprint My_Components:Omron G5V-2-DC12 -> My_Components:Omron G5V-2-H1-DC12
Changed lines of the file:
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@@
 		)
 	)
-	(footprint "My_Components:Omron G5V-2-DC12"
+	(footprint "My_Components:Omron G5V-2-H1-DC12"
 		(layer "F.Cu")
 		(at 152.4 83.82 -90)
-		(descr "Omron relay - DPDT 12VDC 500mW")
+		(descr "Omron relay - DPDT 12VDC 150mW high-sensitivity (G5V-2-H1)")
 		(tags "Relay or Contactor")
 		(property "Reference" "K1"
@@
 			)
 		)
-		(property "Value" "G5V-2 DC12"
+		(property "Value" "G5V-2-H1 DC12"
 			(at 0 0 90)
 			(layer "F.SilkS")
@@
 			)
 		)
-		(property "Datasheet" "G5V-2 DC12"
+		(property "Datasheet" "https://omronfs.omron.com/en_US/ecb/products/pdf/en-g5v_2.pdf"
 			(at 0 0 90)
 			(layer "F.Fab")
@@
 			)
 		)
-		(property "Description" ""
+		(property "Description" "Relay, DPDT (2 Form C), high-sensitivity 12 VDC coil (960 ohm, approx. 150 mW), THT, fully sealed"
 			(at 0 0 90)
 			(layer "F.Fab")
@@
 			)
 		)
-		(property "MFG Part #" "G5V-2-DC12"
+		(property "MFG Part #" "G5V-2-H1 DC12"
 			(at 0 0 90)
 			(layer "F.SilkS")
@@
 			)
 		)
-		(property "JLCPCB Part #" "C28089"
+		(property "JLCPCB Part #" "C128021"
 			(at 0 0 90)
 			(layer "F.SilkS")
@@
 			)
 		)
-		(property ki_fp_filters "RELAY_G5V-2_OMR")
+		(property ki_fp_filters "Omron G5V-2*")
 		(sheetname "/")
 		(sheetfile "Passthrough_HarnessBox_Final.kicad_sch")
