File: PCB Files/Polestar_Flexray.kicad_sch (KiCad schematic)
At the start: 44 parts, among them J1 JAE DX07S024XJ1R1100, J2 Molex 2125280400, J3 JAE MX34032NF4, J4 JAE MX34032NF4, K1 G5V-2-H1 DC12, K2 G5V-2-H1 DC12, Q1 DMN3200U-7, Q2 DMN3200U-7, U1 Vishay DG419LEDY-T1-GE4, U2 Vishay DG419LEDY-T1-GE4, U3 LM53600-Q1, U4 XIAO_RP2350, U5 TJA1082, U6 TJA1082

Commit message: Add CAN-FD controller block, bulk decoupling and FlexRay ERRN wiring
Schematic:
- U8 TCAN4550-Q1 CAN-FD controller with 40 MHz crystal (Y1), SPI link to
  the RP2350, split CAN termination (R17/R18/C23) and nINT pull-up
- C24 10uF on VSUP and C25 10uF on VIO. TI SLLSEZ5D sec 10 requires bulk
  capacitance on both rails in addition to the 100 nF bypass caps
- FlexRay transceiver ERRN outputs wired to the RP2350 (U5.10 -> GP17,
  U6.10 -> GP16) for wake-from-sleep. ERRN is push-pull, no pull-ups needed
- Renamed CAN_* nets to SPI_*/TCAN_*; they are the SPI link to U8, not CAN
- Replaced 12 plain power labels with power symbols, and hid boilerplate
  metadata fields that were rendering on the sheet
- Relay and diode symbol pins retyped from Unspecified to Passive

Netclasses: five colour-coded classes keyed to which side of the MITM cut
a bus sits on (FlexRay car/ECU, CAN car/comma/passthrough). Repaired the
netclass patterns, which all referenced renamed _H/_L nets and matched
nothing, leaving every differential net on Default rules.

Footprints: restored 29 links that Update Symbols from Library had
overwritten, and corrected the Footprint defaults in 14 library symbols so
it cannot recur.

ERC is clean: 0 errors, 0 warnings.

Known issue: C24/C25 placement overlaps U8's courtyard (4 courtyard
overlaps, 6 clearance errors). Board is otherwise unrouted.

Co-Authored-By: Claude Opus 5 <noreply@anthropic.com>
Parts:
- added C13, C14, C23: 4.7nF, Footprints:SAMS CL10B472KB8NNNC, symbol Device:C
- added C17, C18: 2.2pF, Capacitor_SMD:C_0603_1608Metric, symbol Device:C
- added C19: 22uF, Footprints:SAMS CL32B226KAJNNNE, symbol Device:C
- added C20: 470nF, Footprints:SAMS CL10B474KA8NNNC, symbol Device:C
- added C21, C22: 100nF, Footprints:SAMS CL10B104KB8NNNC, symbol Device:C
- added C24: 10uF, Footprints:Taiyo UMK325AB7106KM-P, symbol Device:C
- added C25: 10uF, Footprints:SAMS CL21B106KAYQNNE, symbol Device:C
- added K3: G5V-2-H1 DC12, Footprints:Omron G5V-2-H1-DC12, symbol 2026-08-07_12-56-36:G5V-2_DC12
- added R11, R12, R14, R15: 47, Footprints:Rohm ESR03EZPJ470, symbol Device:R
- added R16, R17, R18: 60R4, Footprints:YAGEO AC0603FR-7W60R4L, symbol Device:R
- added R19: 10K, Footprints:Rohm ESR03EZPJ103, symbol Device:R
- added U8: TCAN4550-Q1, Footprints:TI TCAN4550RGYRQ1, symbol My_Components:TCAN4550-Q1
- added Y1: 40MHz, Crystal:Crystal_SMD_2016-4Pin_2.0x1.6mm, symbol Device:Crystal_GND24
- C12: value 10nF -> 100nF; footprint Footprints:SAMS CL05B103KA5NNNC -> Footprints:SAMS CL10B104KB8NNNC
- C5: footprint Capacitor_SMD:C_0805_2012Metric -> Footprints:SAMS CL21B106KAYQNNE
- C6: footprint Capacitor_SMD:C_1210_3225Metric -> Footprints:Taiyo UMK325AB7106KM-P
- C8: footprint Capacitor_SMD:C_1206_3216Metric -> Footprints:SAMS CL31B475KBHNNNE
- C9: footprint Capacitor_SMD:C_1206_3216Metric -> Footprints:SAMS CL32B226KAJNNNE
- D10, D11: LCSC (none) -> C2905640; MPN (none) -> PESD1FLEX
- K1, K2: footprint Footprints:Omron G5V-2-DC12 -> Footprints:Omron G5V-2-H1-DC12
Connections:
- net +3V3: now also C21.1, C25.1, R19.1, U8.17 (VIO)
- net +5V: no longer C12.1
- net COMMA_N: now also R18.2, U8.10 (CANL)
- net COMMA_P: now also R17.1, U8.11 (CANH)
- net FR_ECU_BM: now also K3.13
- net FR_ECU_BP: now also K3.4
- net FR_RLY_COIL: now also K3.1
- net GND: now also U4.24 (GND), C13.2, C14.2, C17.2, C18.2, C19.2, C20.2, C21.2, C22.2, C23.2, C24.2, C25.2, U8.12 (WAKE), U8.13 (GND), U8.21 (PAD), Y1.2 (G), Y1.4 (G)
- net VIN: now also C12.1, C22.1, C24.1, K3.16, U8.14 (VSUP)
- net FR1_ERRN: now reaches U5.10 (ERRN)
- net FR1_ERRN: now also U4.17 (D13/GP17)
- net TERM_VEH_P: now reaches K2.8
- net TERM_VEH_P: now also R11.1
- net TERM_VEH_N: now reaches K2.9
- net TERM_VEH_N: now also R12.2
- net FR2_ERRN: now reaches U6.10 (ERRN)
- net FR2_ERRN: now also U4.18 (D14/GP16)
- new net: C14.1, R14.2, R15.1
- new net: C13.1, R11.2, R12.1
- new net: C18.1, R16.2, Y1.3
- new net: C23.1, R17.2, R18.1
- new net OSC1: R16.1, U8.1 (OSC1)
- new net OSC2: C17.1, U8.20 (OSC2), Y1.1
- new net SPI_CS: U4.22 (D18/GP9), U8.7 (nCS)
- new net SPI_MISO: U4.20 (D16/GP12), U8.6 (SDO)
- new net SPI_MOSI: U4.19 (D15/GP11), U8.5 (SDI)
- new net SPI_SCLK: U4.21 (D17/GP10), U8.4 (SCLK)
- new net TCAN_FLTR: C20.1, U8.18 (FLTR)
- new net TCAN_RST: U4.16 (D12/GP20), U8.19 (RST)
- new net TCAN_VCC: C19.1, U8.16 (VCCOUT)
- new net TCAN_nINT: R19.2, U4.15 (D11/GP21), U8.8 (nINT)
- new net TERM_ECU_N: K3.9, R15.2
- new net TERM_ECU_P: K3.8, R14.1
- no-connect marks 47 -> 50
Other:
- moved on the sheet: CR2, D10, D11, J4, K2, Q2, R10, R9, U3, U5, U6

Commit message: Add input protection, fix TJA1082 mode strap and Q3 pad mapping
Protection and supply hardening on the only power input, plus three
silent faults found by review.

Input (J2 is the sole feed and sits on constant battery):
- F1 Walter Elec 1206T3A63V, 3A 63V time-lag (LCSC C354897). Previously
  there was no fuse anywhere in the design.
- Q3 reverse-polarity P-FET (DMP4015SSS-13), drain on the fused battery,
  source on VIN, with D14 16V gate clamp and R20 100k pulldown. D9 moved
  to the load side of Q3; as a uni-directional TVS it was forward-biasing
  on a reversed input, and CR1 with it, putting two SMD diodes straight
  across the battery.
- D14 is 16V so it stays off at 14.4V, costing zero standby current.

Q3 pad mapping (would have shipped broken):
- Q3 used a 3-pin generic FET symbol on an 8-pad SOIC-8. KiCad matches pin
  numbers to pad numbers, so gate/drain/source landed on pads 1-3 - all
  three of which are Source on the DMP4015SSS. VBAT_F was shorted to VIN
  through the package and the real gate and drain floated. The board would
  have powered up normally with no reverse protection at all, and ERC does
  not check pad mapping. Fixed with My_Components:DMP4015SSS-13, an 8-pin
  symbol with S on 1-3, G on 4, D on 5-8.

TJA1082 error indication (U5, U6):
- SCSN tied high did not disable SPI. Per datasheet rev 6 sec 6.8 the part
  powers up in SPI mode, where error flags latch until a full 16-bit status
  readout. VIO comes from the XIAO LDO so it rises after VCC, setting UVVIO
  on every power-up, and with SCLK/SDO unconnected nothing could ever clear
  it - ERRN would have latched low forever. Now strapped to simple error
  indication mode: SCSN to GND, SCLK to +3V3.

XIAO supply:
- D12 Schottky + C26 10uF isolating the XIAO 5V pad, which is raw USB VBUS.
  Plugging in USB to flash it previously fought the buck (forced PWM allows
  reverse current) or back-fed VIN through the buck body diode.

DG419 supply and comma-side termination:
- V+ now fed via D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
Parts:
- added C26: 10uF, Footprints:SAMS CL21B106KAYQNNE, symbol Device:C
- added C27: 10nF, Footprints:SAMS CL05B103KA5NNNC, symbol Device:C
- added C28: 100nF, Footprints:SAMS CL10B104KB8NNNC, symbol Device:C
- added D12, D15: DSK14, Footprints:SCHOTTKY - 1A, symbol Device:D_Schottky
- added D13: BZT52C5V1, Footprints:SOD123_DIO, symbol Device:D_Zener
- added D14: BZT52C16, Footprints:SOD123_DIO, symbol Device:D_Zener
- added D16: BZT52C12, Footprints:SOD123_DIO, symbol Device:D_Zener
- added D17: PESD1CAN, Footprints:PESD1CAN, symbol My_Components:PESD1CAN
- added F1: 3A, Footprints:Walter Elec 1206T3A63V, symbol Device:Fuse
- added Q3: DMP4015SSS-13, Package_SO:SOIC-8_3.9x4.9mm_P1.27mm, symbol My_Components:DMP4015SSS-13
- added R20: 100K, Footprints:Rohm ESR03EZPJ104, symbol Device:R
- added R21: 3.3K, Footprints:Rohm ESR03EZPJ332, symbol Device:R
- added R22: 120, Footprints:Rohm ESR03EZPJ121, symbol Device:R
- C17, C18: value 2.2pF -> 2.2pF C0G; footprint Capacitor_SMD:C_0603_1608Metric -> Footprints:FH 0603CG2R2C500NT
- R16: value 60R4 -> 0R; footprint Footprints:YAGEO AC0603FR-7W60R4L -> Footprints:R_0603_1608Metric
- R6: value 1K -> 10K; footprint Footprints:Rohm ESR03EZPJ102 -> Footprints:Rohm ESR03EZPJ103; symbol My_Components:ESR03EZPJ102 -> Device:R
- R8: value 1K -> 3.3K; footprint Footprints:Rohm ESR03EZPJ102 -> Footprints:Rohm ESR03EZPJ332; symbol My_Components:ESR03EZPJ102 -> Device:R
- U3: value LM53600-Q1 -> LM53600LQDSXRQ1; MFG Part # (none) -> LM53600LQDSXRQ1
- Y1: value 40MHz -> 40MHz NX2016SA
Connections:
- net +3V3: now also U5.7 (SCLK), U6.7 (SCLK); no longer U5.9 (SCSN), U6.9 (SCSN)
- net +5V: now also U1.5 (VL), U2.5 (VL), C27.1, D12.2 (A); no longer U4.14 (5V)
- net GND: now also U5.9 (SCSN), U6.9 (SCSN), C26.2, C27.2, C28.2, D13.2 (A), D16.2 (A), D17.3 (CATHODE_COM), R20.2
- net VCU_N_C: now also D17.2 (CATHODE_2)
- net VCU_P_C: now also D17.1 (CATHODE_1), R22.2
- net VIN: now also D14.1 (K), D15.2 (A), Q3.1 (S), Q3.2 (S), Q3.3 (S); no longer J2.4, U1.4 (V+), U1.5 (VL), U2.4 (V+), U2.5 (VL)
- net IGN_GATE: now reaches Q1.1 (G), R6.2, R8.1
- net IGN_GATE: now also D13.1 (K)
- net at U2.8 (NO): now also R22.1
- new net +5V_XIAO: C26.1, D12.1 (K), U4.14 (5V)
- new net Q3_GATE: D14.2 (A), Q3.4 (G), R20.1
- new net SW_IN: D15.1 (K), R21.1
- new net SW_VCC: C28.1, D16.1 (K), R21.2, U1.4 (V+), U2.4 (V+)
- new net VBAT: F1.1, J2.4
- new net VBAT_F: F1.2, Q3.5 (D), Q3.6 (D), Q3.7 (D), Q3.8 (D)
- no-connect marks 50 -> 47
Other:
- moved on the sheet: C1, C10, C11, C12, C13, C14, C17, C18, C19, C2, C20, C21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

Commit message: Re-place board on 98x58 mm outline, add mounting holes and rounded corners
Placement
- Re-placed all 80 footprints to the "wide_2" layout on a 98 x 58 mm
  outline (was 119 x 43 mm). The 5 V buck block (U3, L1, C8-C12, C27,
  R13) and D9/C6 move to the bottom right, the SW_VCC group (D15, R21,
  D16) to the top left, and the comma CAN group (U1, U2, R2, R3, C28)
  shifts left. C11, D9, R13 and R21 also change rotation.
- Pad geometry, sizes, layers and nets verified unchanged across the
  rotations: 389 pads, 126 nets, 0 net changes.

Mechanical
- Added H1-H4: M3, 3.2 mm, non-plated, inset 3.8 mm from both edges.
  Non-plated so enclosure screws do not bond chassis to board ground;
  harness pin 13 is not board GND. PCB-only, no schematic symbols.
- Radiused the four board corners at R3.8 mm. Each arc centre lands on
  its mounting-hole centre, so the corner is concentric with the hole.
- Reshaped the In1.Cu ground pour outline to match the rounded corners
  and dropped its stale square-cornered fill so it repours correctly.

DRC
- Added Polestar_Flexray.kicad_dru. U8 reproduces TI drawing 4225320/A
  (RGY0020A) exactly, which places the exposed pad 0.025 mm from every
  perimeter pin; U3's 0.5 mm-pitch pins sit 0.26 mm apart against a
  0.3 mm Power netclass rule. Both are non-solder-mask-defined, so
  bridging is controlled by the stencil, not copper spacing. The rule
  is scoped to U3/U8 so other footprints are still checked normally.
- Raised U4's reference text from 0.635 mm to 1.0 mm to meet the
  0.8 mm board minimum.
- Now 0 clearance, 0 courtyard-overlap, 0 copper-to-edge and
  0 invalid-outline violations. Remaining items are the 239 unrouted
  ratsnest connections and cosmetic silkscreen warnings.

The board is still unrouted - 0 tracks, 0 vias. Do not fabricate.

Co-Authored-By: Claude Opus 5 <noreply@anthropic.com>
Other:
- moved on the sheet: C1, C10, C11, C12, C13, C14, C17, C18, C19, C2, C20, C23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
